File: hardware/eyeballer-seeker.kicad_sch (KiCad schematic)
At the start: 11 parts, among them SW1 只关雷达, U1 固定 5V, U2 雷达

Commit message: Redraw the system schematic so each wire lands on a pin.
Lay the sheet out left to right from the battery to the radar, move the board into the main area, and export a larger drawing plus a module diagram. ERC reports zero errors.

Co-authored-by: Atraxa <aquaNeosIN@users.noreply.github.com>
Parts:
- removed C1: 100nF, symbol eyeballer:C15
- removed C2: 22uF, symbol eyeballer:C15
- removed C3: 100uF, symbol eyeballer:C30
- removed C4: 100nF, symbol eyeballer:C30
- added C1: 100nF, symbol eyeballer:C_IN
- added C2: 22uF, symbol eyeballer:C_IN
- added C3: 100uF, symbol eyeballer:C_OUT
- added C4: 100nF, symbol eyeballer:C_OUT
- BT1: value 3.7V 锂电 -> 3.7V
- R1, R2: value 220 -> 220Ω
Connections:
- net +5V: now also U1.4 (VOUT), C3.1, C4.1
- net GND: now also A1.2 (GND), A1.9 (GND_J1), BT1.2 (-), U1.3 (GND), U2.2 (GND), C1.2, C2.2, C3.2, C4.2
- net UART1_RX: now also A1.8 (GPIO18)
- net UART1_TX: now also A1.7 (GPIO17)
- net VBAT: now also A1.10 (VBAT1)
- net at SW1.2, U1.1 (VIN): now also U1.2 (EN), C1.1, C2.1
- net at U2.3 (RX): now also R1.1
- net at U2.4 (TX): now also R2.1
Other:
- note added: "1. 从左到右：电池 → 开关 → TPS61023 升压 → 雷达。上面那根 VBAT 是电池正极，同时接到开发板 J1。"
- note added: "2. 雷达 TX 接 H2 脚8（GPIO18，板子接收）。雷达 RX 接 H2 脚7（GPIO17，板子发送）。3.3V，各串 220Ω。"
- note added: "3. 不要把 5V 接到任何 GPIO。脚4和脚5是下载串口。画了叉的脚不接。"
- note added: "4. 升压只从电池取电。排针上的 3.3V 和 VBUS 不能用。VSYS 没有引出来。"
- note added: "5. 开关只关雷达。充电时关掉开关。J1 脚1 = VBAT1，脚2 = GND，插之前用万用表确认。"
- note added: "6. H2 脚序来自官方原理图 PDF（2025-07-28）。另一份说明的脚4到脚8不同，焊前量一下。H2 脚2 的 GND 和下方地线同名，是相连的。"
- note added: "eyeballer-seeker v1 系统接线"
- note removed: "1 同名标号是同一根线。GND：电池负极、升压地、雷达地、H2 脚2、J1 脚2。"
- note removed: "2 雷达串口用 H2 脚7 GPIO17（板子发送）和脚8 GPIO18（板子接收）。3.3V，串联 220 欧。"
- note removed: "3 5V 从电池正极 VBAT1 升压得到。不要用排针上的 3V3，也不要靠 VBUS（只有插着 USB 才有）。"
- note removed: "4 U0TXD，5 U0RXD，6 GPIO16，7 GPIO17，8 GPIO18。HARDWARE_REFERENCE.md 的脚4–8不同，先量再焊。"
- note removed: "4 开关只切断升压模块。电池仍然进 J1，USB 才能充电。充电时把开关关掉。"
- note removed: "5 H2 脚序按 Waveshare 原理图 PDF（2025-07-28）：1 VBUS，2 GND，3 VCC3V3，"
- note removed: "6 J1 在原理图 POWER 区。VBAT1 和 AXP2101 的 BAT（33 脚）是同一网络。"
- note removed: "7 升压模块用固定 5V 的 TPS61023。模块里已有小电容，C1–C4 是线两端再加的。"
- note removed: "AXP2101 的 VSYS（34 脚）没有引到排针或电池座。"
- note removed: "EN 接到 VIN，开关打开模块就工作"
- note removed: "VBAT：电池正极和 J1 脚1。中间没有画成长线，是为了不和别的线叠在一起。"
- note removed: "eyeballer-seeker v1 系统原理图"
- note removed: "不要用脚4 / 脚5 的 UART0，也不要把 5V 碰到任何 GPIO。PA9 本版不接。"
- note removed: "圆屏朝外，雷达天线和屏幕同一面。手静止时让眼睛看路过的人。固件不在这一版。"
- note removed: "接线时读这里"
- note removed: "本图画脚1 = VBAT1、脚2 = GND。插电池前用万用表确认极性。"
- note removed: "雷达 TX 接到 GPIO18，雷达 RX 接到 GPIO17（交叉）"

Commit message: Redraw the schematic in functional blocks and add a first carrier PCB.
Co-authored-by: Atraxa <aquaNeosIN@users.noreply.github.com>
Parts:
- removed A1: 开发板, symbol eyeballer:WS_AMOLED_175
- removed BT1: 3.7V, symbol eyeballer:Battery_1S
- removed C1: 100nF, symbol eyeballer:C_IN
- removed C2: 22uF, symbol eyeballer:C_IN
- removed C3: 100uF, symbol eyeballer:C_OUT
- removed C4: 100nF, symbol eyeballer:C_OUT
- removed R1, R2: 220Ω, symbol eyeballer:R_H
- removed SW1: 只关雷达, symbol eyeballer:SW_Slide
- removed U1: 固定 5V, symbol eyeballer:TPS61023_MOD
- removed U2: 雷达, symbol eyeballer:LD2450
- added BT1: Li-ion 3.7V, symbol eyeballer:Battery_Cell
- added C1, C4: 100nF, Capacitor_SMD:C_0805_2012Metric, symbol eyeballer:C
- added C2: 22uF, Capacitor_SMD:C_0805_2012Metric, symbol eyeballer:C
- added C3: 100uF, Capacitor_SMD:C_1206_3216Metric, symbol eyeballer:C
- added J1: MX1.25, Connector_JST:JST_GH_SM02B-GHS-TB_1x02-1MP_P1.25mm_Horizontal, symbol eyeballer:Conn_01x02_Socket
- added J2: to board J1, Connector_PinHeader_2.54mm:PinHeader_1x02_P2.54mm_Vertical, symbol eyeballer:Conn_01x02_Pin
- added J3: TPS61023 module, Connector_PinHeader_2.54mm:PinHeader_1x04_P2.54mm_Vertical, symbol eyeballer:Conn_01x04_Socket
- added J4: HLK-LD2450, Connector_PinHeader_2.54mm:PinHeader_1x04_P2.54mm_Vertical, symbol eyeballer:Conn_01x04_Pin
- added J5: to H2, Connector_PinHeader_2.54mm:PinHeader_1x08_P2.54mm_Vertical, symbol eyeballer:Conn_01x08_Socket
- added R1, R2: 220, Resistor_SMD:R_0805_2012Metric, symbol eyeballer:R
- added SW1: SPDT, Button_Switch_SMD:SW_SPDT_CK_JS102011SAQN, symbol eyeballer:SW_SPDT
Connections:
- net GND: now also BT1.2 (-), C1.2, C2.2, C3.2, C4.2, J1.2 (Pin_2), J2.2 (Pin_2), J3.2 (Pin_2), J4.2 (Pin_2), J5.2 (Pin_2)
- net VBAT: now also BT1.1 (+), J1.1 (Pin_1), J2.1 (Pin_1), SW1.2 (B)
- new net: J4.3 (Pin_3), R2.1
- new net: J4.4 (Pin_4), R1.1
- new net +5V_RADAR: C3.1, C4.1, J3.4 (Pin_4), J4.1 (Pin_1)
- new net BOOST_IN: C1.1, C2.1, J3.1 (Pin_1), J3.3 (Pin_3), SW1.1 (A)
- new net RADAR_RX: J5.7 (Pin_7), R1.2
- new net RADAR_TX: J5.8 (Pin_8), R2.2
Other:
- note added: "1 5V"
- note added: "1 VBUS"
- note added: "2 GND"
- note added: "3 TX"
- note added: "3 VCC3V3"
- note added: "4 RX"
- note added: "4 U0TXD GPIO43"
- note added: "5 U0RXD GPIO44"
- note added: "5V boost TPS61023"
- note added: "6 GPIO16"
- note added: "7 GPIO17 radar RX"
- note added: "8 GPIO18 radar TX"
- note added: "Battery and switch"
- note added: "Battery connector J1"
- note added: "ESP32-S3 board header H2"
- note added: "J1 接电池。J2 接到开发板电池座，和板内充电并联。"
- note added: "RADAR_TX：雷达 TX 到 H2 脚 8。RADAR_RX：H2 脚 7 到雷达 RX。焊前用万用表核对脚序和电池正负。"
- note added: "Radar HLK-LD2450"
- note added: "同名网络是连在一起的：VBAT、GND、+5V_RADAR、BOOST_IN、RADAR_TX、RADAR_RX。"
- note added: "排针脚序来自 Waveshare 原理图 PDF（2025-07-28）。"
- note added: "电池正极是 VBAT。开关脚 2 是公共端，只给升压；脚 3 不接。"
- note added: "脚序 1 VIN、2 GND、3 EN、4 VOUT，以模块实物为准。EN 与 VIN 同网。"
- note added: "脚序 1=5V 2=GND 3=TX 4=RX。PA9 不接。串口 3.3V，各串 220Ω。"
- note removed: "1. 从左到右：电池 → 开关 → TPS61023 升压 → 雷达。上面那根 VBAT 是电池正极，同时接到开发板 J1。"
- note removed: "2. 雷达 TX 接 H2 脚8（GPIO18，板子接收）。雷达 RX 接 H2 脚7（GPIO17，板子发送）。3.3V，各串 220Ω。"
- note removed: "3. 不要把 5V 接到任何 GPIO。脚4和脚5是下载串口。画了叉的脚不接。"
- note removed: "4. 升压只从电池取电。排针上的 3.3V 和 VBUS 不能用。VSYS 没有引出来。"
- note removed: "5. 开关只关雷达。充电时关掉开关。J1 脚1 = VBAT1，脚2 = GND，插之前用万用表确认。"
- note removed: "6. H2 脚序来自官方原理图 PDF（2025-07-28）。另一份说明的脚4到脚8不同，焊前量一下。H2 脚2 的 GND 和下方地线同名，是相连的。"
- note removed: "eyeballer-seeker v1 系统接线"
- title: eyeballer-seeker v1 system wiring -> eyeballer-seeker v1
